Commit message: fixing initial commit

File: dorna_description/urdf/dorna.urdf (robot description, URDF)
Before this commit: robot dorna, 10 links, 9 joints
Links:
- link dorna_end_effector: geometry collision mesh filename=package://dorna_description/meshes/one_finger_asm.stl scale=0.001 0.001 0.001; visual mesh filename=package://dorna_description/meshes/one_finger_asm.stl scale=0.001 0.001 0.001
Joints:
- joint dorna_arm_4_to_dorna_end_effector: origin xyz=0.0315 0.0 0.0 rpy=0 0 -1.57079632679 -> xyz=0.0315 0.0 0.0 rpy=0 -1.57079632679 1.57079632679
- joint fixed: origin xyz=0 0 0.76 rpy=0 0 0 -> xyz=0 0 0 rpy=0 0 0

File: dorna_description/urdf/dorna.urdf.xacro (robot description, xacro)
@@ -1,4 +1,6 @@
 <?xml version="1.0"?>
 <robot name="dorna" xmlns:xacro="http://ros.org/wiki/xacro">
+  <xacro:arg name="stand_alone" default="true" /> <!-- true = position controller; false = effort controller -->
+  <xacro:property name="stand_alone" value="$(arg stand_alone)"/>
   <xacro:macro name="dorna" params="parent *base_origin">
     <!-- ############################## -->
@@ -22,5 +24,5 @@
     </xacro:property>
     <xacro:property name="dorna_base_color">
-      <material name="orange"/>
+      <material name="black"/>
     </xacro:property>
     <xacro:property name="dorna_base_origin">
@@ -118,5 +120,5 @@
     </xacro:property>
     <xacro:property name="dorna_arm_3_color">
-      <material name="orange"/>
+      <material name="red"/>
     </xacro:property>
     <xacro:property name="dorna_arm_3_origin">
@@ -141,5 +143,5 @@
     </xacro:property>
     <xacro:property name="dorna_arm_4_color">
-      <material name="orange"/>
+      <material name="red"/>
     </xacro:property>
     <xacro:property name="dorna_arm_4_origin">
@@ -167,9 +169,10 @@
     </xacro:property>
     <xacro:property name="dorna_end_effector_origin">
-      <origin xyz="0 0 0" rpy="0 ${-PI/2} 0"/>
+      <origin xyz="0 0 0" rpy="0 0 0"/>
     </xacro:property>
     <xacro:property name="dorna_end_effector_mesh">
       <geometry>
-        <mesh filename="package://dorna_description/meshes/1_finger_tool.stl" scale="${0.001} ${0.001} ${0.001}"/>
+        <mesh filename="package://dorna_description/meshes/one_finger_asm.stl" scale="${0.001} ${0.001} ${0.001}"/>
+        <!-- <mesh filename="package://dorna_description/meshes/1_finger_tool.stl" scale="${0.001} ${0.001} ${0.001}"/> -->
       </geometry>
     </xacro:property>
@@ -308,5 +311,5 @@
       <parent link="dorna_arm_4"/>
       <child link="dorna_end_effector"/>
-      <origin xyz="0.0315 0.0 0.0" rpy="0 0 ${-PI/2}"/>
+      <origin xyz="0.0315 0.0 0.0" rpy="0 ${-PI/2} ${PI/2}"/>
     </joint>
     <xacro:link_block prt_name="dorna_end_effector">
@@ -355,3 +358,10 @@
     </gazebo>
   </xacro:macro>
+  <xacro:if value="${stand_alone}">
+    <link name="world">
+    </link>
+    <xacro:dorna parent="world">
+      <origin xyz="0 0 0" rpy="0 0 0"/>
+    </xacro:dorna>
+  </xacro:if>
 </robot>
